File: my-kkeb/Git_pad.kicad_sch (KiCad schematic)
At the start: 36 parts, among them J9 Conn_01x04, SW3 RotaryEncoder_Switch, SW4 RotaryEncoder_Switch, U4 MCP23017x-x-SO

Commit message: This is basically the finished thing. The only thing left if the BOM
Parts:
- added C7: 100nF, Capacitor_SMD:C_0603_1608Metric, symbol Device:C
- added C8: 10uF, Capacitor_SMD:C_0805_2012Metric, symbol Device:C
- added R11, R12: 100, Resistor_SMD:R_0603_1608Metric, symbol Device:R
- J9: footprint Connector_PinHeader_2.54mm:PinHeader_1x04_P2.54mm_Vertical -> CUSTOM:PogoMag_1x04_P2.54mm_RightAngle
- MX100, MX101, MX102, MX103, MX104, MX105, MX106, MX107, MX108, MX109, MX110, MX111, MX112, MX97, MX98, MX99: footprint PCM_marbastlib-mx:SW_MX_HS_CPG151101S11_1u -> CUSTOM:SW_MX_HS_CPG151101S11_1u_PinSwap
Connections:
- net Type_C_GND: now also C7.2, C8.2
- net Type_C_SCL: now also R12.1; no longer U4.12 (SCK)
- net Type_C_SDA: now also R11.1; no longer U4.13 (SDA)
- net Type_C_VCC: now also C7.1, C8.1
- new net: R12.2, U4.12 (SCK)
- new net: R11.2, U4.13 (SDA)
