File: my-kkeb/Left.kicad_sch (KiCad schematic)
At the start: 63 parts, among them J5 Type_C, J6 Conn_01x04, SW2 RotaryEncoder_Switch

Commit message: This is basically the finished thing. The only thing left if the BOM
Parts:
- added R1, R2: 2.2k, Resistor_SMD:R_0603_1608Metric, symbol Device:R
- added U7: ER_OLEDM0.91_1x-I2C, Display:ER_OLEDM0.91_1x-I2C, symbol Display_Graphic:ER_OLEDM0.91_1x-I2C
- J5: footprint CUSTOM:USB_C_Receptacle_HRO_TYPE-C-31-M-12_4Pin -> CUSTOM:USB_C_Receptacle_HRO_TYPE-C-31-M-12_4Pin_Fixed
- J6: footprint Connector_PinHeader_2.54mm:PinHeader_1x04_P2.54mm_Vertical -> CUSTOM:PogoMag_1x04_P2.54mm_RightAngle
- MX1, MX10, MX11, MX12, MX13, MX14, MX15, MX16, MX17, MX18, MX19, MX2, MX20, MX21, MX22, MX23, MX24, MX25, MX26, MX27, MX28, MX29, MX3, MX4, MX5, MX6, MX7, MX8, MX9: footprint PCM_marbastlib-mx:SW_MX_HS_CPG151101S11_1u -> CUSTOM:SW_MX_HS_CPG151101S11_1u_PinSwap
Connections:
- net Type_C_GND: now also U7.1 (GND)
- net Type_C_SCL: now also R1.1, U7.3 (SCL)
- net Type_C_SDA: now also R2.1, U7.4 (SDA)
- net Type_C_VCC: now also R1.2, R2.2, U7.2 (VCC)
Other:
- moved on the sheet: J5
