File: my-kkeb/Macro_pad.kicad_sch (KiCad schematic)
At the start: 36 parts, among them J7 Conn_01x04, J8 Conn_01x04, U3 MCP23017x-x-SO, U6 ER_OLEDM0.91_1x-I2C

Commit message: This is basically the finished thing. The only thing left if the BOM
Parts:
- added C5: 100nF, Capacitor_SMD:C_0603_1608Metric, symbol Device:C
- added C6: 10uF, Capacitor_SMD:C_0805_2012Metric, symbol Device:C
- added R10, R9: 100, Resistor_SMD:R_0603_1608Metric, symbol Device:R
- J7, J8: footprint Connector_PinHeader_2.54mm:PinHeader_1x04_P2.54mm_Vertical -> CUSTOM:PogoMag_1x04_P2.54mm_RightAngle
- MX81, MX82, MX83, MX84, MX85, MX86, MX87, MX88, MX89, MX90, MX91, MX92, MX93, MX94, MX95, MX96: footprint PCM_marbastlib-mx:SW_MX_HS_CPG151101S11_1u -> CUSTOM:SW_MX_HS_CPG151101S11_1u_PinSwap
Connections:
- net Type_C_GND: now also C5.2, C6.2
- net Type_C_SCL: now also R10.1; no longer U3.12 (SCK)
- net Type_C_SDA: now also R9.1; no longer U3.13 (SDA)
- net Type_C_VCC: now also C5.1, C6.1
- new net: R10.2, U3.12 (SCK)
- new net: R9.2, U3.13 (SDA)
