File: my-kkeb/Numpad.kicad_sch (KiCad schematic)
At the start: 47 parts, among them J3 Conn_01x04, U2 MCP23017x-x-SO

Commit message: This is basically the finished thing. The only thing left if the BOM
Parts:
- added C3: 100nF, Capacitor_SMD:C_0603_1608Metric, symbol Device:C
- added C4: 10uF, Capacitor_SMD:C_0805_2012Metric, symbol Device:C
- added D113: 1N4148, Diode_THT:D_DO-35_SOD27_P7.62mm_Horizontal, symbol Diode:1N4148
- added MX113: MX_SW_HS, CUSTOM:SW_MX_HS_CPG151101S11_1u_PinSwap, symbol PCM_marbastlib-mx:MX_SW_HS_CPG151101S11
- added R7, R8: 100, Resistor_SMD:R_0603_1608Metric, symbol Device:R
- J3: footprint Connector_PinHeader_2.54mm:PinHeader_1x04_P2.54mm_Vertical -> CUSTOM:PogoMag_1x04_P2.54mm_RightAngle
- MX59, MX60, MX61, MX62, MX63, MX64, MX65, MX66, MX67, MX68, MX69, MX70, MX71, MX72, MX73, MX74, MX75, MX76, MX77, MX78, MX79, MX80: footprint PCM_marbastlib-mx:SW_MX_HS_CPG151101S11_1u -> CUSTOM:SW_MX_HS_CPG151101S11_1u_PinSwap
Connections:
- net Numpad_COL_2: now also MX113.1
- net Numpad_ROW_4: now also D113.1 (K)
- net Type_C_GND: now also C3.2, C4.2
- net Type_C_SCL: now also R8.1; no longer U2.12 (SCK)
- net Type_C_SDA: now also R7.1; no longer U2.13 (SDA)
- net Type_C_VCC: now also C3.1, C4.1
- new net: R8.2, U2.12 (SCK)
- new net: D113.2 (A), MX113.2
- new net: R7.2, U2.13 (SDA)
