File: my-kkeb/Right.kicad_sch (KiCad schematic)
At the start: 64 parts, among them J11 TypeC, J4 Conn_01x04, SW1 RotaryEncoder_Switch, U1 MCP23017x-x-SO, U5 ER_OLEDM0.91_1x-I2C

Commit message: This is basically the finished thing. The only thing left if the BOM
Parts:
- added C1: 100nF, Capacitor_SMD:C_0603_1608Metric, symbol Device:C
- added C2: 10uF, Capacitor_SMD:C_0805_2012Metric, symbol Device:C
- added R3, R4: 100, Resistor_SMD:R_0603_1608Metric, symbol Device:R
- J11: footprint CUSTOM:USB_C_Receptacle_HRO_TYPE-C-31-M-12_4Pin -> CUSTOM:USB_C_Receptacle_HRO_TYPE-C-31-M-12_4Pin_Fixed
- J4: footprint Connector_PinHeader_2.54mm:PinHeader_1x04_P2.54mm_Vertical -> CUSTOM:PogoMag_1x04_P2.54mm_RightAngle
- MX30, MX31, MX32, MX33, MX34, MX35, MX36, MX37, MX38, MX39, MX40, MX41, MX42, MX43, MX44, MX45, MX46, MX47, MX48, MX49, MX50, MX51, MX52, MX53, MX54, MX55, MX56, MX57, MX58: footprint PCM_marbastlib-mx:SW_MX_HS_CPG151101S11_1u -> CUSTOM:SW_MX_HS_CPG151101S11_1u_PinSwap
Connections:
- net Type_C_GND: now also C1.2, C2.2
- net Type_C_SCL: now also R3.1; no longer U1.12 (SCK)
- net Type_C_SDA: now also R4.1; no longer U1.13 (SDA)
- net Type_C_VCC: now also C1.1, C2.1
- new net: R3.2, U1.12 (SCK)
- new net: R4.2, U1.13 (SDA)
