File: my-kkeb/my-kkeb.kicad_pcb (KiCad board)
At the start: 2 copper layers, 247 parts, among them J10 USB_C_Receptacle, J11 TypeC, J3 Conn_01x04, J4 Conn_01x04, J5 Type_C, J6 Conn_01x04, J7 Conn_01x04, J8 Conn_01x04, J9 Conn_01x04, SW1 RotaryEncoder_Switch, SW2 RotaryEncoder_Switch, SW3 RotaryEncoder_Switch, SW4 RotaryEncoder_Switch, U1 MCP23017x-x-SO, U2 MCP23017x-x-SO, U3 MCP23017x-x-SO, U4 MCP23017x-x-SO, U5 ER_OLEDM0.91_1x-I2C, U6 ER_OLEDM0.91_1x-I2C

Commit message: This is basically the finished thing. The only thing left if the BOM
Parts:
- removed J10: USB_C_Receptacle, Connector_USB:USB_C_Receptacle_HRO_TYPE-C-31-M-12
- added C1: 100nF, Capacitor_SMD:C_0603_1608Metric, B.Cu at (280.2, -66.8)
- added C2: 10uF, Capacitor_SMD:C_0805_2012Metric, B.Cu at (276.6, -66.9)
- added C3: 100nF, Capacitor_SMD:C_0603_1608Metric, B.Cu at (411.8, -47.1)
- added C4: 10uF, Capacitor_SMD:C_0805_2012Metric, B.Cu at (409.7, -51.5)
- added C5: 100nF, Capacitor_SMD:C_0603_1608Metric, B.Cu at (-122.9, -176.5)
- added C6: 10uF, Capacitor_SMD:C_0805_2012Metric, B.Cu at (-118.8, -176.5)
- added C7: 100nF, Capacitor_SMD:C_0603_1608Metric, B.Cu at (-210.5, -179.3)
- added C8: 10uF, Capacitor_SMD:C_0805_2012Metric, B.Cu at (-206.5, -179.2)
- added D113: 1N4148, Diode_THT:D_DO-35_SOD27_P7.62mm_Horizontal, B.Cu at (468.2, -65.9)
- added MX113: MX_SW_HS, CUSTOM:SW_MX_HS_CPG151101S11_1u_PinSwap, B.Cu at (476.2, -73.6)
- added R1: 2.2k, Resistor_SMD:R_0603_1608Metric, B.Cu at (-18.4, -101.8)
- added R10: 100, Resistor_SMD:R_0603_1608Metric, B.Cu at (-127.8, -161.7)
- added R11: 100, Resistor_SMD:R_0603_1608Metric, B.Cu at (-198.3, -179.0)
- added R12: 100, Resistor_SMD:R_0603_1608Metric, B.Cu at (-202.3, -179.0)
- added R2: 2.2k, Resistor_SMD:R_0603_1608Metric, B.Cu at (-22.3, -101.7)
- added R3: 100, Resistor_SMD:R_0603_1608Metric, B.Cu at (274.6, -73.2)
- added R4: 100, Resistor_SMD:R_0603_1608Metric, B.Cu at (284.0, -66.8)
- added R7: 100, Resistor_SMD:R_0603_1608Metric, B.Cu at (425.2, -38.2)
- added R8: 100, Resistor_SMD:R_0603_1608Metric, B.Cu at (429.7, -42.3)
- added R9: 100, Resistor_SMD:R_0603_1608Metric, B.Cu at (-127.8, -165.4)
- added REF**: MountingHole_2.2mm_M2, MountingHole:MountingHole_2.2mm_M2, F.Cu at (428.5, -140.5)
- added REF**: MountingHole_2.2mm_M2, MountingHole:MountingHole_2.2mm_M2, F.Cu at (337.4, -96.0)
- added REF**: MountingHole_2.2mm_M2, MountingHole:MountingHole_2.2mm_M2, F.Cu at (227.3, -76.0)
- added REF**: MountingHole_2.2mm_M2, MountingHole:MountingHole_2.2mm_M2, F.Cu at (19.0, -77.0)
- added REF**: MountingHole_2.2mm_M2, MountingHole:MountingHole_2.2mm_M2, F.Cu at (339.0, -147.0)
- added REF**: MountingHole_2.2mm_M2, MountingHole:MountingHole_2.2mm_M2, F.Cu at (357.2, -138.0)
- added REF**: MountingHole_2.2mm_M2, MountingHole:MountingHole_2.2mm_M2, F.Cu at (-246.0, -171.5)
- added REF**: MountingHole_2.2mm_M2, MountingHole:MountingHole_2.2mm_M2, F.Cu at (-47.6, -138.0)
- added REF**: MountingHole_2.2mm_M2, MountingHole:MountingHole_2.2mm_M2, F.Cu at (-169.5, -88.5)
- added REF**: MountingHole_2.2mm_M2, MountingHole:MountingHole_2.2mm_M2, F.Cu at (-34.5, -158.5)
- added REF**: MountingHole_2.2mm_M2, MountingHole:MountingHole_2.2mm_M2, F.Cu at (-168.0, -108.0)
- added REF**: MountingHole_2.2mm_M2, MountingHole:MountingHole_2.2mm_M2, F.Cu at (-133.3, -138.0)
- added REF**: MountingHole_2.2mm_M2, MountingHole:MountingHole_2.2mm_M2, F.Cu at (447.5, -102.0)
- added REF**: MountingHole_2.2mm_M2, MountingHole:MountingHole_2.2mm_M2, F.Cu at (304.9, -77.0)
- added REF**: MountingHole_2.2mm_M2, MountingHole:MountingHole_2.2mm_M2, F.Cu at (483.5, -20.0)
- added REF**: MountingHole_2.2mm_M2, MountingHole:MountingHole_2.2mm_M2, F.Cu at (-133.5, -108.0)
- added REF**: MountingHole_2.2mm_M2, MountingHole:MountingHole_2.2mm_M2, F.Cu at (9.00, -121.0)
- added REF**: MountingHole_2.2mm_M2, MountingHole:MountingHole_2.2mm_M2, F.Cu at (353.0, -106.0)
- added REF**: MountingHole_2.2mm_M2, MountingHole:MountingHole_2.2mm_M2, F.Cu at (466.5, -140.5)
- added REF**: MountingHole_2.2mm_M2, MountingHole:MountingHole_2.2mm_M2, F.Cu at (412.0, -20.0)
- added REF**: MountingHole_2.2mm_M2, MountingHole:MountingHole_2.2mm_M2, F.Cu at (96.5, -76.0)
- added REF**: MountingHole_2.2mm_M2, MountingHole:MountingHole_2.2mm_M2, F.Cu at (47.0, -126.0)
- added REF**: MountingHole_2.2mm_M2, MountingHole:MountingHole_2.2mm_M2, F.Cu at (314.9, -121.0)
- added REF**: MountingHole_2.2mm_M2, MountingHole:MountingHole_2.2mm_M2, F.Cu at (-71.5, -102.0)
- added REF**: MountingHole_2.2mm_M2, MountingHole:MountingHole_2.2mm_M2, F.Cu at (-128.5, -102.5)
- added REF**: MountingHole_2.2mm_M2, MountingHole:MountingHole_2.2mm_M2, F.Cu at (-169.5, -170.5)
- added REF**: MountingHole_2.2mm_M2, MountingHole:MountingHole_2.2mm_M2, F.Cu at (-49.0, -108.0)
- added REF**: MountingHole_2.2mm_M2, MountingHole:MountingHole_2.2mm_M2, F.Cu at (404.8, -138.0)
- added REF**: MountingHole_2.2mm_M2, MountingHole:MountingHole_2.2mm_M2, F.Cu at (-71.5, -140.5)
- added REF**: MountingHole_2.2mm_M2, MountingHole:MountingHole_2.2mm_M2, F.Cu at (-166.7, -138.0)
- added REF**: MountingHole_2.2mm_M2, MountingHole:MountingHole_2.2mm_M2, F.Cu at (-56.0, -169.5)
- added REF**: MountingHole_2.2mm_M2, MountingHole:MountingHole_2.2mm_M2, F.Cu at (-13.5, -96.0)
- added REF**: MountingHole_2.2mm_M2, MountingHole:MountingHole_2.2mm_M2, F.Cu at (-228.5, -101.0)
- added REF**: MountingHole_2.2mm_M2, MountingHole:MountingHole_2.2mm_M2, F.Cu at (-33.3, -138.0)
- added REF**: MountingHole_2.2mm_M2, MountingHole:MountingHole_2.2mm_M2, F.Cu at (258.5, -111.5)
- added U7: ER_OLEDM0.91_1x-I2C, Display:ER_OLEDM0.91_1x-I2C, F.Cu at (-15.2, -104.8)
- A1, D1, D10, D100, D101, D102, D103, D104, D105, D106, D107, D108, D109, D11, D110, D111, D112, D12, D13, D14, D15, D16, D17, D18, D19, D2, D20, D21, D22, D23, D24, D25, D26, D27, D28, D29, D3, D30, D31, D32, D33, D34, D35, D36, D37, D38, D39, D4, D40, D41, D42, D43, D44, D45, D46, D47, D48, D49, D5, D50, D51, D52, D53, D54, D55, D56, D57, D58, D59, D6, D60, D61, D62, D63, D64, D65, D66, D67, D68, D69, D7, D70, D71, D72, D73, D74, D75, D76, D77, D78, D79, D8, D80, D81, D82, D83, D84, D85, D86, D87, D88, D89, D9, D90, D91, D92, D93, D94, D95, D96, D97, D98, D99, U1, U2, U3, U4: moved to B.Cu
- J11, J5: footprint CUSTOM:USB_C_Receptacle_HRO_TYPE-C-31-M-12_4Pin -> CUSTOM:USB_C_Receptacle_HRO_TYPE-C-31-M-12_4Pin_Fixed; moved to B.Cu
- J3, J6, J7: footprint Connector_PinHeader_2.54mm:PinHeader_1x04_P2.54mm_Vertical -> CUSTOM:PogoMag_1x04_P2.54mm_RightAngle_Mirror
- J4, J8, J9: footprint Connector_PinHeader_2.54mm:PinHeader_1x04_P2.54mm_Vertical -> CUSTOM:PogoMag_1x04_P2.54mm_RightAngle
- MX1, MX10, MX100, MX101, MX102, MX103, MX104, MX105, MX106, MX107, MX108, MX109, MX11, MX110, MX111, MX112, MX12, MX13, MX14, MX15, MX16, MX17, MX18, MX19, MX2, MX20, MX21, MX22, MX23, MX24, MX25, MX26, MX27, MX28, MX29, MX3, MX30, MX31, MX32, MX33, MX34, MX35, MX36, MX37, MX38, MX39, MX4, MX40, MX41, MX42, MX43, MX44, MX45, MX46, MX47, MX48, MX49, MX5, MX50, MX51, MX52, MX53, MX54, MX55, MX56, MX57, MX58, MX59, MX6, MX60, MX61, MX62, MX63, MX64, MX65, MX66, MX67, MX68, MX69, MX7, MX70, MX71, MX72, MX73, MX74, MX75, MX76, MX77, MX78, MX79, MX8, MX80, MX81, MX82, MX83, MX84, MX85, MX86, MX87, MX88, MX89, MX9, MX90, MX91, MX92, MX93, MX94, MX95, MX96, MX97, MX98, MX99: footprint PCM_marbastlib-mx:SW_MX_HS_CPG151101S11_1u -> CUSTOM:SW_MX_HS_CPG151101S11_1u_PinSwap; moved to B.Cu
- moved U3 531.3 mm to (-116.5, -168.8), turned to 90 degrees
- moved J7 506.7 mm to (-133.5, -126.0)
- moved U6 478.0 mm to (-98.5, -165.1), turned to 90 degrees
- moved D81 471.0 mm to (-127.3, -142.1), turned to 90 degrees
- moved D85 467.5 mm to (-127.3, -123.0), turned to 90 degrees
- moved D89 466.7 mm to (-129.3, -106.0), turned to 90 degrees
- moved D82 461.0 mm to (-108.1, -142.1), turned to 90 degrees
- moved D93 460.4 mm to (-127.3, -84.9), turned to 90 degrees
- moved J8 458.9 mm to (-47.5, -126.0)
- moved D97 458.4 mm to (-246.4, -139.9), turned to 90 degrees
- moved D86 457.3 mm to (-108.1, -123.0), turned to 90 degrees
- moved D98 453.9 mm to (-246.4, -120.8), turned to 90 degrees
- moved D90 453.7 mm to (-108.1, -104.0), turned to 90 degrees
- moved D83 451.8 mm to (-89.0, -142.1), turned to 90 degrees
- moved MX70 451.7 mm to (476.2, -111.7), turned to 180 degrees
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Connections:
- A1 pad 1: /Left/Type_C_SDA -> /Git_pad/Type_C_SDA
- A1 pad 13: /Left/Type_C_GND -> /Git_pad/Type_C_GND
- A1 pad 18: /Left/Type_C_GND -> /Git_pad/Type_C_GND
- A1 pad 2: /Left/Type_C_SCL -> /Git_pad/Type_C_SCL
- A1 pad 23: /Left/Type_C_GND -> /Git_pad/Type_C_GND
- A1 pad 28: /Left/Type_C_GND -> /Git_pad/Type_C_GND
- A1 pad 3: /Left/Type_C_GND -> /Git_pad/Type_C_GND
- A1 pad 38: /Left/Type_C_GND -> /Git_pad/Type_C_GND
- A1 pad 8: /Left/Type_C_GND -> /Git_pad/Type_C_GND
- J11 pad 1: /Left/Type_C_SDA -> /Git_pad/Type_C_SDA
- J11 pad 2: /Left/Type_C_SCL -> /Git_pad/Type_C_SCL
- J11 pad 4: /Left/Type_C_GND -> /Git_pad/Type_C_GND
- J3 pad 1: /Numpad/Type_C_SDA -> /Git_pad/Type_C_SDA
- J3 pad 2: /Numpad/Type_C_SCL -> /Git_pad/Type_C_SCL
- J3 pad 3: /Numpad/Type_C_VCC -> /Git_pad/Type_C_VCC
- J3 pad 4: /Numpad/Type_C_GND -> /Git_pad/Type_C_GND
- J4 pad 1: /Left/Type_C_SDA -> /Git_pad/Type_C_SDA
- J4 pad 2: /Left/Type_C_SCL -> /Git_pad/Type_C_SCL
- J4 pad 4: /Left/Type_C_GND -> /Git_pad/Type_C_GND
- J5 pad 1: /Left/Type_C_SDA -> /Git_pad/Type_C_SDA
- J5 pad 2: /Left/Type_C_SCL -> /Git_pad/Type_C_SCL
- J5 pad 4: /Left/Type_C_GND -> /Git_pad/Type_C_GND
- J6 pad 1: /Left/Type_C_SDA -> /Git_pad/Type_C_SDA
- J6 pad 2: /Left/Type_C_SCL -> /Git_pad/Type_C_SCL
- J6 pad 4: /Left/Type_C_GND -> /Git_pad/Type_C_GND
- SW1 pad C: /Left/Type_C_GND -> /Git_pad/Type_C_GND
- SW1 pad S1: /Left/Type_C_GND -> /Git_pad/Type_C_GND
- SW2 pad C: /Left/Type_C_GND -> /Git_pad/Type_C_GND
- SW2 pad S1: /Left/Type_C_GND -> /Git_pad/Type_C_GND
- U1 pad 10: /Left/Type_C_GND -> /Git_pad/Type_C_GND
- U1 pad 12: /Left/Type_C_SDA -> Net-(U1-SCK)
- U1 pad 13: /Left/Type_C_SCL -> Net-(U1-SDA)
- U1 pad 15: unconnected-(U1-A0-Pad15) -> /Git_pad/Type_C_VCC
- U1 pad 16: unconnected-(U1-A1-Pad16) -> /Git_pad/Type_C_GND
- U1 pad 17: unconnected-(U1-A2-Pad17) -> /Git_pad/Type_C_GND
- U1 pad 18: unconnected-(U1-~{RESET}-Pad18) -> /Git_pad/Type_C_VCC
- U2 pad 10: /Numpad/Type_C_GND -> /Git_pad/Type_C_GND
- U2 pad 12: /Numpad/Type_C_SCL -> Net-(U2-SCK)
- U2 pad 13: /Numpad/Type_C_SDA -> Net-(U2-SDA)
- U2 pad 15: unconnected-(U2-A0-Pad15) -> /Git_pad/Type_C_VCC
- U2 pad 16: unconnected-(U2-A1-Pad16) -> /Git_pad/Type_C_VCC
- U2 pad 17: unconnected-(U2-A2-Pad17) -> /Git_pad/Type_C_GND
- U2 pad 18: unconnected-(U2-~{RESET}-Pad18) -> /Git_pad/Type_C_VCC
- U2 pad 9: /Numpad/Type_C_VCC -> /Git_pad/Type_C_VCC
- U3 pad 12: /Git_pad/Type_C_SDA -> Net-(U3-SCK)
- U3 pad 13: /Git_pad/Type_C_SCL -> Net-(U3-SDA)
- U3 pad 15: unconnected-(U3-A0-Pad15) -> /Git_pad/Type_C_GND
- U3 pad 16: unconnected-(U3-A1-Pad16) -> /Git_pad/Type_C_GND
- U3 pad 17: unconnected-(U3-A2-Pad17) -> /Git_pad/Type_C_VCC
- U3 pad 18: unconnected-(U3-~{RESET}-Pad18) -> /Git_pad/Type_C_VCC
- U4 pad 12: /Git_pad/Type_C_SDA -> Net-(U4-SCK)
- U4 pad 13: /Git_pad/Type_C_SCL -> Net-(U4-SDA)
- U4 pad 15: unconnected-(U4-A0-Pad15) -> /Git_pad/Type_C_GND
- U4 pad 16: unconnected-(U4-A1-Pad16) -> /Git_pad/Type_C_VCC
- U4 pad 17: unconnected-(U4-A2-Pad17) -> /Git_pad/Type_C_VCC
- U4 pad 18: unconnected-(U4-~{RESET}-Pad18) -> /Git_pad/Type_C_VCC
- U5 pad 1: /Left/Type_C_GND -> /Git_pad/Type_C_GND
- U5 pad 3: /Left/Type_C_SCL -> /Git_pad/Type_C_SCL
- U5 pad 4: /Left/Type_C_SDA -> /Git_pad/Type_C_SDA
Routing:
- net /Git_pad/Type_C_GND: track 0.00 -> 1215.0 mm, vias 0 -> 36
- net /Git_pad/Type_C_VCC: track 0.00 -> 984.4 mm, vias 0 -> 23
- net /Git_pad/Type_C_SCL: track 0.00 -> 861.3 mm, vias 0 -> 21
- net /Git_pad/Type_C_SDA: track 0.00 -> 848.4 mm, vias 0 -> 17
- net /Right/Right_ROW_0: track 0.00 -> 254.7 mm, vias 0 -> 5
- net /Left/Left_COL_0: track 0.00 -> 248.6 mm, vias 0 -> 5
- net /Right/Right_COL_4: track 0.00 -> 234.1 mm, vias 0 -> 3
- net /Left/Left_ROW_4: track 0.00 -> 221.3 mm, vias 0 -> 10
- net /Left/Left_ROW_3: track 0.00 -> 215.6 mm, vias 0 -> 12
- net /Macro_pad/Mac_ROW_3: track 0.00 -> 208.0 mm, vias 0 -> 2
- net /Numpad/Numpad_ROW_0: track 0.00 -> 206.6 mm, vias 0 -> 9
- net /Right/Right_COL_3: track 0.00 -> 205.0 mm, vias 0 -> 4
- net /Right/Right_ROW_1: track 0.00 -> 204.5 mm, vias 0 -> 4
- net /Git_pad/Git_ROW_3: track 0.00 -> 203.5 mm, vias 0 -> 3
- net /Left/Left_ROW_5: track 0.00 -> 197.8 mm, vias 0 -> 6
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Other:
- board outline added: 739.3 x 173.1 mm
